File: beaverworksGit.kicad_sch (KiCad schematic)
At the start: 2 parts, among them J1 Analog, J2 Digital

Commit message: First prototype
Parts:
- removed J1: Analog, Connector_PinHeader_2.54mm:PinHeader_1x15_P2.54mm_Vertical, symbol Connector_Generic:Conn_01x15
- removed J2: Digital, Connector_PinHeader_2.54mm:PinHeader_1x15_P2.54mm_Vertical, symbol Connector_Generic:Conn_01x15
- added A1: ARDUINO_MEGA_2560_REV3_A000067, ARDUINO_MEGA_2560_REV3_A000067:ARDUINO_ARDUINO_MEGA_2560_REV3_A000067, symbol ARDUINO_MEGA_2560_REV3_A000067:ARDUINO_MEGA_2560_REV3_A000067
- added BT1: Battery, symbol Device:Battery
- added D1: LED, symbol Device:LED
- added M1: Motor_Servo, symbol Motor:Motor_Servo
- added M2, M3, M4, M5: Motor_DC, symbol Motor:Motor_DC
- added R1: R, symbol Device:R
- added U1: MPU-6050, Sensor_Motion:InvenSense_QFN-24_4x4mm_P0.5mm, symbol Sensor_Motion:MPU-6050
- added U2: DHT11, Sensor:Aosong_DHT11_5.5x12.0_P2.54mm, symbol Sensor:DHT11
- added U3: (no value), symbol Audio:Sound_Sensor_Elegoo
- added U4: HC-SR04, HC-SR04:XCVR_HC-SR04, symbol HC-SR04:HC-SR04
- added U5: L298N, Package_TO_SOT_THT:TO-220-15_P2.54x5.08mm_StaggerOdd_Lead4.58mm_Vertical, symbol Driver_Motor:L298N
Connections:
- new net: M2.1 (+), M3.1 (+), U5.13 (OUT3)
- new net: M2.2 (-), M3.2 (-), U5.14 (OUT4)
- new net: A1.17, U5.10 (IN3)
- new net: A1.6, U5.11 (EnB)
- new net: A1.16, U5.12 (IN4)
- new net: M4.1 (+), M5.1 (+), U5.2 (OUT1)
- new net: M4.2 (-), M5.2 (-), U5.3 (OUT2)
- new net: BT1.1 (+), U5.4 (Vs)
- new net: A1.20, U5.5 (IN1)
- new net: A1.7, U5.6 (EnA)
- new net: A1.19, U5.7 (IN2)
- new net: A1.GND5, BT1.2 (-), U2.4 (GND), U3. (GND), U5.8 (GND)
- new net: A1.5V_2 (+5V_2), M1.2 (+), U1.13 (VDD), U1.8 (VLOGIC), U2.1 (VDD), U3. (GND), U4.1 (VCC), U5.9 (Vss)
- new net: A1.24, U1.23 (SCL)
- new net: A1.22, U1.24 (SDA)
- new net: D1.1 (K), R1.1
- new net: A1.GND3, M1.3 (-), R1.2, U4.4 (GND)
- new net: A1.3, U4.2 (TRIG)
- new net: A1.4, U4.3 (ECHO)
- new net: A1.5, M1.1 (PWM)
- new net: A1.AD2, U2.2 (DATA)
- new net: A1.8, D1.2 (A)
